Commit message: Fixing erros

File: hans_t30_description/urdf/hans_module.urdf.xacro (robot description, xacro)
@@ -2,5 +2,4 @@
 <robot xmlns:xacro="http://ros.org/wiki/xacro"
        name="robotiq_hande" >
-  <!-- robotiq hande_gripper -->
   <xacro:include filename="$(find hans_t30_description)/urdf/hans_t30.urdf.xacro" />
   <xacro:hans30 prefix=""/>

File: hans_t30_description/urdf/hans_t30.urdf.xacro (robot description, xacro)
@@ -95,6 +95,6 @@
       </link>
       <joint name="motor1" type="revolute">
-        <origin xyz="-0.12 0 0" rpy="0 ${-PI/2} 0" />
-        <parent link="elfin_module_14" />
+        <origin xyz="-0.12 0 0" rpy="0 ${-3.1416/2} 0" />
+        <parent link="motor1_link" />
         <child link="dummy_link1" />
         <axis xyz="0 0 1" />
@@ -102,9 +102,14 @@
       </joint>
       <joint name="motor2" type="revolute">
-        <origin xyz="0 -0.16 0" rpy="${PI/2} 0 0" />
-        <parent link="elfin_module_14" />
+        <origin xyz="0 -0.16 0" rpy="${3.1416/2} 0 0" />
+        <parent link="motor1_link" />
         <child link="dummy_link2" />
         <axis xyz="0 0 1" />
         <limit lower="-3.14" upper="3.14" effort="34" velocity="1.57" />
+      </joint>
+      <joint name="${prefix}motor1_cover_joint" type="fixed">
+        <origin rpy="0 0 0" xyz="0 0 0.0"/>
+        <parent link="${prefix}motor1_link"/>
+        <child link="${prefix}motor1_cover"/>
       </joint>
       <gazebo>

File: hans_t49_description/urdf/hans_module.urdf.xacro (robot description, xacro)
@@ -2,5 +2,4 @@
 <robot xmlns:xacro="http://ros.org/wiki/xacro"
        name="robotiq_hande" >
-  <!-- robotiq hande_gripper -->
   <xacro:include filename="$(find hans_t49_description)/urdf/hans_t49.urdf.xacro" />
   <xacro:hans49 prefix=""/>

File: hans_t49_description/urdf/hans_t49.urdf.xacro (robot description, xacro)
@@ -95,6 +95,6 @@
       </link>
       <joint name="motor1" type="revolute">
-        <origin xyz="-0.12 0 0" rpy="0 ${-PI/2} 0" />
-        <parent link="elfin_module_14" />
+        <origin xyz="-0.12 0 0" rpy="0 ${-3.1416/2} 0" />
+        <parent link="motor1_link" />
         <child link="dummy_link1" />
         <axis xyz="0 0 1" />
@@ -102,9 +102,14 @@
       </joint>
       <joint name="motor2" type="revolute">
-        <origin xyz="0 -0.16 0" rpy="${PI/2} 0 0" />
-        <parent link="elfin_module_14" />
+        <origin xyz="0 -0.16 0" rpy="${3.1416/2} 0 0" />
+        <parent link="motor1_link" />
         <child link="dummy_link2" />
         <axis xyz="0 0 1" />
         <limit lower="-3.14" upper="3.14" effort="34" velocity="1.57" />
+      </joint>
+      <joint name="${prefix}motor1_cover_joint" type="fixed">
+        <origin rpy="0 0 0" xyz="0 0 0.0"/>
+        <parent link="${prefix}motor1_link"/>
+        <child link="${prefix}motor1_cover"/>
       </joint>
       <gazebo>

File: hans_t9_4_description/urdf/hans_module.urdf.xacro (robot description, xacro)
@@ -2,7 +2,6 @@
 <robot xmlns:xacro="http://ros.org/wiki/xacro"
        name="robotiq_hande" >
-  <!-- robotiq hande_gripper -->
-  <xacro:include filename="$(find hans_t9.4_description)/urdf/hans_t9.4.urdf.xacro" />
-  <xacro:hans9.4 prefix=""/>
+  <xacro:include filename="$(find hans_t9_4_description)/urdf/hans_t9.4.urdf.xacro" />
+  <xacro:hans9_4 prefix=""/>
   <link name="world" />
   <joint name="world_to_hande_joint" type="fixed">

File: hans_t9_4_description/urdf/hans_t9.4.urdf.xacro (robot description, xacro)
@@ -1,5 +1,5 @@
 <?xml version="1.0"?>
 <robot xmlns:xacro="http://ros.org/wiki/xacro">
-  <xacro:macro name="hans9.4" params="prefix">
+  <xacro:macro name="hans9_4" params="prefix">
       <link name="${prefix}motor1_link">
         <inertial>
@@ -95,6 +95,6 @@
       </link>
       <joint name="motor1" type="revolute">
-        <origin xyz="-0.12 0 0" rpy="0 ${-PI/2} 0" />
-        <parent link="elfin_module_14" />
+        <origin xyz="-0.12 0 0" rpy="0 ${-3.1416/2} 0" />
+        <parent link="motor1_link" />
         <child link="dummy_link1" />
         <axis xyz="0 0 1" />
@@ -102,9 +102,14 @@
       </joint>
       <joint name="motor2" type="revolute">
-        <origin xyz="0 -0.16 0" rpy="${PI/2} 0 0" />
-        <parent link="elfin_module_14" />
+        <origin xyz="0 -0.16 0" rpy="${3.1416/2} 0 0" />
+        <parent link="motor1_link" />
         <child link="dummy_link2" />
         <axis xyz="0 0 1" />
         <limit lower="-3.14" upper="3.14" effort="34" velocity="1.57" />
+      </joint>
+      <joint name="${prefix}motor1_cover_joint" type="fixed">
+        <origin rpy="0 0 0" xyz="0 0 0.0"/>
+        <parent link="${prefix}motor1_link"/>
+        <child link="${prefix}motor1_cover"/>
       </joint>
       <gazebo>
