Commit message: Fixing URDFs

File: hans_t30_description/urdf/hans_t30.urdf (robot description, URDF)
Before this commit: robot robotiq_hande, 5 links, 4 joints
Links:
- link motor1_cover: geometry collision mesh filename=package://hans_t30_description/meshes/HANS_T30_Black.dae scale=0.001 0.001 0.001; visual mesh filename=package://hans_t30_description/meshes/HANS_T30_Black.dae scale=0.001 0.001 0.001
Joints:
- joint motor1: origin xyz=-0.12 0 0 rpy=0 -1.5708 0 -> xyz=-0.109255 0 0.149255 rpy=0 -1.5708 0
- joint motor2: origin xyz=0 -0.16 0 rpy=1.5708 0 0 -> xyz=0 0 0 rpy=0 -1.5708 0

File: hans_t30_description/urdf/hans_t30.urdf.xacro (robot description, xacro)
@@ -37,5 +37,5 @@
           <origin rpy="0 0 0" xyz="0 0 0"/>
           <geometry>
-            <mesh filename="package://hans_t30_description/meshes/HANS_T30_black.dae" scale="0.001 0.001 0.001"/>
+            <mesh filename="package://hans_t30_description/meshes/HANS_T30_Black.dae" scale="0.001 0.001 0.001"/>
           </geometry>
           <material name="Gazebo/Black">
@@ -46,5 +46,5 @@
           <origin rpy="0 0 0" xyz="0 0 0"/>
           <geometry>
-            <mesh filename="package://hans_t30_description/meshes/HANS_T30_black.dae" scale="0.001 0.001 0.001"/>
+            <mesh filename="package://hans_t30_description/meshes/HANS_T30_Black.dae" scale="0.001 0.001 0.001"/>
           </geometry>
         </collision>
@@ -95,5 +95,5 @@
       </link>
       <joint name="motor1" type="revolute">
-        <origin xyz="-0.12 0 0" rpy="0 ${-3.1416/2} 0" />
+        <origin rpy="0 -1.5708 0" xyz="-0.109255 0 0.149255"/>
         <parent link="motor1_link" />
         <child link="dummy_link1" />
@@ -102,5 +102,5 @@
       </joint>
       <joint name="motor2" type="revolute">
-        <origin xyz="0 -0.16 0" rpy="${3.1416/2} 0 0" />
+        <origin rpy="0 -1.5708 0" xyz="0 0 0"/>
         <parent link="motor1_link" />
         <child link="dummy_link2" />

File: hans_t49_description/urdf/hans_t49.urdf (robot description, URDF)
Before this commit: robot robotiq_hande, 5 links, 4 joints
Links:
- link motor1_cover: geometry collision mesh filename=package://hans_t49_description/meshes/HANS_T49_Black.dae scale=0.001 0.001 0.001; visual mesh filename=package://hans_t49_description/meshes/HANS_T49_Black.dae scale=0.001 0.001 0.001
Joints:
- joint motor1: origin xyz=-0.12 0 0 rpy=0 -1.5708 0 -> xyz=0.109255 0 0.16074 rpy=0 -1.5708 0
- joint motor2: origin xyz=0 -0.16 0 rpy=1.5708 0 0 -> xyz=0 0 0 rpy=1.5708 0 0

File: hans_t49_description/urdf/hans_t49.urdf.xacro (robot description, xacro)
@@ -37,5 +37,5 @@
           <origin rpy="0 0 0" xyz="0 0 0"/>
           <geometry>
-            <mesh filename="package://hans_t49_description/meshes/HANS_T49_black.dae" scale="0.001 0.001 0.001"/>
+            <mesh filename="package://hans_t49_description/meshes/HANS_T49_Black.dae" scale="0.001 0.001 0.001"/>
           </geometry>
           <material name="Gazebo/Black">
@@ -46,5 +46,5 @@
           <origin rpy="0 0 0" xyz="0 0 0"/>
           <geometry>
-            <mesh filename="package://hans_t49_description/meshes/HANS_T49_black.dae" scale="0.001 0.001 0.001"/>
+            <mesh filename="package://hans_t49_description/meshes/HANS_T49_Black.dae" scale="0.001 0.001 0.001"/>
           </geometry>
         </collision>
@@ -95,5 +95,5 @@
       </link>
       <joint name="motor1" type="revolute">
-        <origin xyz="-0.12 0 0" rpy="0 ${-3.1416/2} 0" />
+        <origin rpy="0 -1.5708 0" xyz="0.109255 0 0.16074"/>
         <parent link="motor1_link" />
         <child link="dummy_link1" />
@@ -102,5 +102,5 @@
       </joint>
       <joint name="motor2" type="revolute">
-        <origin xyz="0 -0.16 0" rpy="${3.1416/2} 0 0" />
+        <origin rpy="1.5708 0 0" xyz="0 0 0"/>
         <parent link="motor1_link" />
         <child link="dummy_link2" />

File: hans_t9_4_description/urdf/hans_t9.4.urdf (robot description, URDF)
Before this commit: robot robotiq_hande, 5 links, 4 joints
Links:
- link motor1_cover: geometry collision mesh filename=package://hans_t9_4_description/meshes/HANS_T5.4_black.dae scale=0.001 0.001 0.001; visual mesh filename=package://hans_t9_4_description/meshes/HANS_T5.4_black.dae scale=0.001 0.001 0.001
- link motor1_link: geometry collision mesh filename=package://hans_t9_4_description/meshes/HANS_T5.4.dae scale=0.001 0.001 0.001; visual mesh filename=package://hans_t9_4_description/meshes/HANS_T5.4.dae scale=0.001 0.001 0.001
Joints:
- joint motor1: origin xyz=-0.12 0 0 rpy=0 -1.5708 0 -> xyz=-0.10625569 0 0.14675569 rpy=0 -1.5708 0
- joint motor2: origin xyz=0 -0.16 0 rpy=1.5708 0 0 -> xyz=0 0 0 rpy=0 1.5708 0

File: hans_t9_4_description/urdf/hans_t9.4.urdf.xacro (robot description, xacro)
@@ -11,5 +11,5 @@
           <origin rpy="0 0 0" xyz="0 0 0"/>
           <geometry>
-            <mesh filename="package://hans_t49_description/meshes/HANS_T49.dae" scale="0.001 0.001 0.001"/>
+            <mesh filename="package://hans_t9_4_description/meshes/HANS_T5.4.dae" scale="0.001 0.001 0.001"/>
           </geometry>
           <material name="Gazebo/White">
@@ -20,5 +20,5 @@
           <origin rpy="0 0 0" xyz="0 0 0"/>
           <geometry>
-            <mesh filename="package://hans_t49_description/meshes/HANS_T49.dae" scale="0.001 0.001 0.001"/>
+            <mesh filename="package://hans_t9_4_description/meshes/HANS_T5.4.dae" scale="0.001 0.001 0.001"/>
           </geometry>
         </collision>
@@ -37,5 +37,5 @@
           <origin rpy="0 0 0" xyz="0 0 0"/>
           <geometry>
-            <mesh filename="package://hans_t49_description/meshes/HANS_T49_black.dae" scale="0.001 0.001 0.001"/>
+            <mesh filename="package://hans_t9_4_description/meshes/HANS_T5.4_black.dae" scale="0.001 0.001 0.001"/>
           </geometry>
           <material name="Gazebo/Black">
@@ -46,5 +46,5 @@
           <origin rpy="0 0 0" xyz="0 0 0"/>
           <geometry>
-            <mesh filename="package://hans_t49_description/meshes/HANS_T49_black.dae" scale="0.001 0.001 0.001"/>
+            <mesh filename="package://hans_t9_4_description/meshes/HANS_T5.4_black.dae" scale="0.001 0.001 0.001"/>
           </geometry>
         </collision>
@@ -95,5 +95,5 @@
       </link>
       <joint name="motor1" type="revolute">
-        <origin xyz="-0.12 0 0" rpy="0 ${-3.1416/2} 0" />
+        <origin rpy="0 -1.5708 0" xyz="-0.10625569 0 0.14675569"/>
         <parent link="motor1_link" />
         <child link="dummy_link1" />
@@ -102,5 +102,5 @@
       </joint>
       <joint name="motor2" type="revolute">
-        <origin xyz="0 -0.16 0" rpy="${3.1416/2} 0 0" />
+        <origin rpy="0 1.5708 0" xyz="0 0 0"/>
         <parent link="motor1_link" />
         <child link="dummy_link2" />

Commit message: Fixing rotation axis

File: hans_t30_description/urdf/hans_t30.urdf (robot description, URDF)
Before this commit: robot robotiq_hande, 5 links, 4 joints
Joints:
- joint motor1: axis 0 0 1 -> 1 0 0

File: hans_t30_description/urdf/hans_t30.urdf.xacro (robot description, xacro)
@@ -98,5 +98,5 @@
         <parent link="motor1_link" />
         <child link="dummy_link1" />
-        <axis xyz="0 0 1" />
+        <axis xyz="1 0 0"/>
         <limit lower="-3.14" upper="3.14" effort="34" velocity="1.57" />
       </joint>

File: hans_t49_description/urdf/hans_t49.urdf (robot description, URDF)
Before this commit: robot robotiq_hande, 5 links, 4 joints
Joints:
- joint motor2: axis 0 0 1 -> 0 1 0

File: hans_t49_description/urdf/hans_t49.urdf.xacro (robot description, xacro)
@@ -105,5 +105,5 @@
         <parent link="motor1_link" />
         <child link="dummy_link2" />
-        <axis xyz="0 0 1" />
+        <axis xyz="0 1 0" />
         <limit lower="-3.14" upper="3.14" effort="34" velocity="1.57" />
       </joint>

File: hans_t9_4_description/urdf/hans_t9.4.urdf (robot description, URDF)
Before this commit: robot hans9_4, 5 links, 4 joints
Joints:
- joint motor1: axis 0 0 1 -> 1 0 0

File: hans_t9_4_description/urdf/hans_t9.4.urdf.xacro (robot description, xacro)
@@ -98,5 +98,5 @@
         <parent link="motor1_link" />
         <child link="dummy_link1" />
-        <axis xyz="0 0 1" />
+        <axis xyz="1 0 0" />
         <limit lower="-3.14" upper="3.14" effort="34" velocity="1.57" />
       </joint>
